File: parts/oomp_project_github_hanqaqa_easyduino_raspberry_pi_pico_2040_current/data/oomp_design/Easyduino_RP2040.kicad_sch (KiCad schematic)
At the start: 65 parts, among them J1 USB_C_Receptacle_USB2.0, J3 Conn_01x20, J4 Conn_01x20, J5 Conn_01x03, J6 Conn_01x03_MountingPin, SW1 SW_Push, SW2 SW_Push, U1 XC6206P332MR, U2 RP2040, U3 W25Q16JVUXIQ, Y1 12MHz

Commit message: changes
Parts:
- J3, J4: symbol Connector_Generic:Conn_01x20 -> OOMP:electronic_connector_header_2_54_mm_pitch_through_hole_20_pin
- J5: footprint Connector_PinHeader_2.54mm:PinHeader_1x03_P2.54mm_Vertical -> OOMP_MachineSolder:electronic_connector_header_2_54_mm_pitch_through_hole_3_pin; symbol Connector_Generic:Conn_01x03 -> OOMP:electronic_connector_header_2_54_mm_pitch_through_hole_3_pin

Commit message: current
Parts:
- D1: footprint Diode_SMD:D_SOD-123 -> OOMP_MachineSolder:electronic_diode_schottky_sod_123_ss14; symbol Device:D_Schottky -> OOMP:electronic_diode_schottky_sod_123_ss14
- SW1, SW2: symbol Switch:SW_Push -> OOMP:electronic_switch_tactile_surface_mount_xunpu_ts_1088_ar02016
