File: parts/oomp_project_github_hanqaqa_easyduino_raspberry_pi_pico_2040_current/data/oomp_design/Easyduino_RP2040.kicad_sch (KiCad schematic)
At the start: 65 parts, among them J1 USB_C_Receptacle_USB2.0, J3 Conn_01x20, J4 Conn_01x20, J5 Conn_01x03, J6 Conn_01x03_MountingPin, SW1 SW_Push, SW2 SW_Push, U1 XC6206P332MR, U2 RP2040, U3 W25Q16JVUXIQ, Y1 12MHz

Commit message: working
Parts:
- D1: footprint OOMP_MachineSolder:electronic_diode_schottky_sod_123_ss14 -> Diode_SMD:D_SOD-123
- D2, D3, D4: footprint OOMP_MachineSolder:electronic_led_0402 -> LED_SMD:LED_0402_1005Metric; symbol OOMP:electronic_led_0402 -> OOMP:electronic_led_0402_blue
- J5: footprint OOMP_MachineSolder:electronic_connector_header_2_54_mm_pitch_through_hole_3_pin -> Connector_PinHeader_2.54mm:PinHeader_1x03_P2.54mm_Vertical
- U1: symbol Regulator_Linear:XC6206PxxxMR -> OOMP:electronic_ic_sot_23_power_management_linear_voltage_regulator_3_3_volt_torex_xc6206p332mr
