File: parts/oomp_project_github_hanqaqa_easyduino_stm32f103_bluepill_current/data/oomp_design/Easyduino_STM32F103.kicad_sch (KiCad schematic)
At the start: 30 parts, among them J1 USB_C_Receptacle_USB2.0, J2 Conn_01x20, J3 Conn_01x20, J4 Conn_01x04, SW1 SW_Push, SW2 SW_Push, U1 XC6206P332MR, U2 STM32F103C8Tx, Y1 8MHz, Y2 32.768kHz

Commit message: changes
Parts:
- J2, J3: symbol Connector_Generic:Conn_01x20 -> OOMP:electronic_connector_header_2_54_mm_pitch_through_hole_20_pin
- J4: symbol Connector_Generic:Conn_01x04 -> OOMP:electronic_connector_header_2_54_mm_pitch_through_hole_4_pin
- Y1: footprint Crystal:Crystal_SMD_5032-2Pin_5.0x3.2mm -> OOMP_MachineSolder:electronic_crystal_5032_surface_mount_2_pin_8_mhz_20_pf; symbol Device:Crystal -> OOMP:electronic_crystal_5032_surface_mount_2_pin_8_mhz_20_pf
- Y2: footprint Crystal:Crystal_SMD_3215-2Pin_3.2x1.5mm -> OOMP_MachineSolder:electronic_crystal_3215_surface_mount_2_pin_32_768_khz_12_5_pf; symbol Device:Crystal -> OOMP:electronic_crystal_3215_surface_mount_2_pin_32_768_khz_12_5_pf

Commit message: current
Parts:
- SW1, SW2: symbol Switch:SW_Push -> OOMP:electronic_switch_tactile_surface_mount_xunpu_ts_1088_ar02016
