File: parts/oomp_project_github_hanqaqa_easyduino_stm32f103_bluepill_current/data/oomp_design/Easyduino_STM32F103.kicad_sch (KiCad schematic)
At the start: 30 parts, among them J1 USB_C_Receptacle_USB2.0, J2 Conn_01x20, J3 Conn_01x20, J4 Conn_01x04, SW1 SW_Push, SW2 SW_Push, U1 XC6206P332MR, U2 STM32F103C8Tx, Y1 8MHz, Y2 32.768kHz

Commit message: working
Parts:
- D1, D2: footprint OOMP_MachineSolder:electronic_led_0402 -> LED_SMD:LED_0402_1005Metric; symbol OOMP:electronic_led_0402 -> OOMP:electronic_led_0402_blue
- U1: symbol Regulator_Linear:XC6206PxxxMR -> OOMP:electronic_ic_sot_23_power_management_linear_voltage_regulator_3_3_volt_torex_xc6206p332mr
- Y1: footprint OOMP_MachineSolder:electronic_crystal_5032_surface_mount_2_pin_8_mhz_20_pf -> Crystal:Crystal_SMD_5032-2Pin_5.0x3.2mm
- Y2: footprint OOMP_MachineSolder:electronic_crystal_3215_surface_mount_2_pin_32_768_khz_12_5_pf -> Crystal:Crystal_SMD_3215-2Pin_3.2x1.5mm
