File: parts/oomp_project_github_hanqaqa_easyduino_stm32f103_bluepill_current/data/oomp_design/Easyduino_STM32F103.kicad_pcb (KiCad board)
At the start: 4 copper layers, 23 x 53 mm, 30 parts, among them J1 USB_C_Receptacle_USB2.0, J2 Conn_01x20, J3 Conn_01x20, J4 Conn_01x04, SW1 SW_Push, SW2 SW_Push, U1 XC6206P332MR, U2 STM32F103C8Tx, Y1 8MHz, Y2 32.768kHz

Commit message: changes
Parts:
- C10, C11, C7, C8: footprint Capacitor_SMD:C_0402_1005Metric -> OOMP_MachineSolder:electronic_capacitor_0402_18_pico_farad
- Y1: footprint Crystal:Crystal_SMD_5032-2Pin_5.0x3.2mm -> OOMP_MachineSolder:electronic_crystal_5032_surface_mount_2_pin_8_mhz_20_pf
- Y2: footprint Crystal:Crystal_SMD_3215-2Pin_3.2x1.5mm -> OOMP_MachineSolder:electronic_crystal_3215_surface_mount_2_pin_32_768_khz_12_5_pf

Commit message: working
Parts:
- C10, C11, C7, C8: footprint OOMP_MachineSolder:electronic_capacitor_0402_18_pico_farad -> Capacitor_SMD:C_0402_1005Metric
- D1, D2: footprint OOMP_MachineSolder:electronic_led_0402 -> LED_SMD:LED_0402_1005Metric
- R2: footprint OOMP_MachineSolder:electronic_resistor_0402_5100_ohm -> Resistor_SMD:R_0402_1005Metric
- R3: footprint OOMP_MachineSolder:electronic_resistor_0402_10000_ohm -> Resistor_SMD:R_0402_1005Metric
- R6, R7: footprint OOMP_MachineSolder:electronic_resistor_0402_1000_ohm -> Resistor_SMD:R_0402_1005Metric
- Y1: footprint OOMP_MachineSolder:electronic_crystal_5032_surface_mount_2_pin_8_mhz_20_pf -> Crystal:Crystal_SMD_5032-2Pin_5.0x3.2mm
- Y2: footprint OOMP_MachineSolder:electronic_crystal_3215_surface_mount_2_pin_32_768_khz_12_5_pf -> Crystal:Crystal_SMD_3215-2Pin_3.2x1.5mm
