File: parts/oomp_project_github_hanqaqa_easyduino_atmega328p_arduino_nano_current/data/oomp_design/Easyduino_Atmega_Nano.kicad_sch (KiCad schematic)
At the start: 31 parts, among them J1 USB_C_Receptacle_USB2.0, J2 ICSP, SW1 SW_Push, U1 ATmega328P-A, U2 XC6206P502MR, U3 CP2102N-Axx-xQFN28, Y1 16 MHz

Commit message: changes
Parts:
- Y1: symbol Device:Crystal_GND24 -> OOMP:electronic_crystal_3225_surface_mount_4_pin_16_mhz_20_pf
Changed lines of the file:
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@@
   (symbol (lib_id "power:GND") (at 147.32 46.99 0) (unit 1) (body_style 1) (exclude_from_sim no) (in_bom yes) (on_board yes) (in_pos_files yes) (dnp no) (fields_autoplaced yes) (property "Reference" "#PWR023" (at 147.32 53.34 0) (hide yes) (show_name no) (do_not_autoplace no) (effects (font (size 1.27 1.27)))) (property "Value" "GND" (at 147.32 52.07 0) (show_name no) (do_not_autoplace no) (effects (font (size 1.27 1.27)))) (property "Footprint" "" (at 147.32 46.99 0) (hide yes) (show_name no) (do_not_autoplace no) (effects (font (size 1.27 1.27)))) (property "Datasheet" "" (at 147.32 46.99 0) (hide yes) (show_name no) (do_not_autoplace no) (effects (font (size 1.27 1.27)))) (property "Description" "" (at 147.32 46.99 0) (show_name no) (do_not_autoplace no) (effects (font (size 1.27 1.27)))) (pin "1") (instances (project "Easyduino_Atmega_Nano" (path "/8ab39f15-d4dc-4110-b18a-e9bac4395ea8" (reference "#PWR023") (unit 1)))))
   (symbol (lib_id "Device:R") (at 64.77 53.34 90) (unit 1) (body_style 1) (exclude_from_sim no) (in_bom yes) (on_board yes) (in_pos_files yes) (dnp no) (property "Reference" "R2" (at 62.23 55.88 90) (show_name no) (do_not_autoplace no) (effects (font (size 1.27 1.27)))) (property "Value" "5.1k" (at 67.31 55.88 90) (show_name no) (do_not_autoplace no) (effects (font (size 1.27 1.27)))) (property "Footprint" "Resistor_SMD:R_0402_1005Metric" (at 64.77 55.118 90) (hide yes) (show_name no) (do_not_autoplace no) (effects (font (size 1.27 1.27)))) (property "Datasheet" "" (at 64.77 53.34 0) (hide yes) (show_name no) (do_not_autoplace no) (effects (font (size 1.27 1.27)))) (property "Description" "" (at 64.77 53.34 0) (show_name no) (do_not_autoplace no) (effects (font (size 1.27 1.27)))) (property "LCSC" "C25905" (at 64.77 53.34 0) (hide yes) (show_name no) (do_not_autoplace no) (effects (font (size 1.27 1.27)))) (pin "1") (pin "2") (instances (project "Easyduino_Atmega_Nano" (path "/8ab39f15-d4dc-4110-b18a-e9bac4395ea8" (reference "R2") (unit 1)))))
-  (symbol (lib_id "Device:Crystal_GND24") (at 251.46 87.63 0) (unit 1) (body_style 1) (exclude_from_sim no) (in_bom yes) (on_board yes) (in_pos_files yes) (dnp no) (property "Reference" "Y1" (at 269.875 82.55 0) (show_name no) (do_not_autoplace no) (effects (font (size 1.27 1.27)))) (property "Value" "16 MHz" (at 269.875 85.09 0) (show_name no) (do_not_autoplace no) (effects (font (size 1.27 1.27)))) (property "Footprint" "Crystal:Crystal_SMD_3225-4Pin_3.2x2.5mm" (at 251.46 87.63 0) (hide yes) (show_name no) (do_not_autoplace no) (effects (font (size 1.27 1.27)))) (property "Datasheet" "" (at 251.46 87.63 0) (hide yes) (show_name no) (do_not_autoplace no) (effects (font (size 1.27 1.27)))) (property "Description" "Four pin crystal, GND on pins 2 and 4" (at 251.46 87.63 0) (hide yes) (show_name no) (do_not_autoplace no) (effects (font (size 1.27 1.27)))) (property "LCSC" "C13738" (at 251.46 87.63 0) (hide yes) (show_name no) (do_not_autoplace no) (effects (font (size 1.27 1.27)))) (pin "1") (pin "2") (pin "3") (pin "4") (instances (project "Easyduino_Atmega_Nano" (path "/8ab39f15-d4dc-4110-b18a-e9bac4395ea8" (reference "Y1") (unit 1)))))
+  (symbol (lib_id "OOMP:electronic_crystal_3225_surface_mount_4_pin_16_mhz_20_pf") (at 251.46 87.63 0) (unit 1) (body_style 1) (exclude_from_sim no) (in_bom yes) (on_board yes) (in_pos_files yes) (dnp no) (property "Reference" "Y1" (at 269.875 82.55 0) (show_name no) (do_not_autoplace no) (effects (font (size 1.27 1.27)))) (property "Value" "16 MHz" (at 269.875 85.09 0) (show_name no) (do_not_autoplace no) (effects (font (size 1.27 1.27)))) (property "Footprint" "Crystal:Crystal_SMD_3225-4Pin_3.2x2.5mm" (at 251.46 87.63 0) (hide yes) (show_name no) (do_not_autoplace no) (effects (font (size 1.27 1.27)))) (property "Datasheet" "" (at 251.46 87.63 0) (hide yes) (show_name no) (do_not_autoplace no) (effects (font (size 1.27 1.27)))) (property "Description" "Four pin crystal, GND on pins 2 and 4" (at 251.46 87.63 0) (hide yes) (show_name no) (do_not_autoplace no) (effects (font (size 1.27 1.27)))) (property "LCSC" "C13738" (at 251.46 87.63 0) (hide yes) (show_name no) (do_not_autoplace no) (effects (font (size 1.27 1.27)))) (pin "1") (pin "2") (pin "3") (pin "4") (instances (project "Easyduino_Atmega_Nano" (path "/8ab39f15-d4dc-4110-b18a-e9bac4395ea8" (reference "Y1") (unit 1)))))
   (sheet (at 218.44 173.355) (size 24.765 3.81) (exclude_from_sim no) (in_bom yes) (on_board yes) (dnp no) (fields_autoplaced yes) (stroke (width 0.1524) (type solid)) (fill (color 0 0 0 0)) (property "Sheetname" "References" (at 218.44 172.2784 0) (show_name no) (do_not_autoplace no) (effects (font (size 2 2) (bold yes)) (justify left bottom))) (property "Sheetfile" "References.kicad_sch" (at 218.44 177.7496 0) (show_name no) (do_not_autoplace no) (effects (font (size 1.27 1.27)) (justify left top))) (instances (project "Easyduino_Atmega_Nano" (path "/8ab39f15-d4dc-4110-b18a-e9bac4395ea8" (page "2")))))
   (sheet_instances (path "/" (page "1")))

Commit message: current
Parts:
- F1: footprint Fuse:Fuse_0402_1005Metric -> OOMP_MachineSolder:electronic_fuse_0402_resettable; symbol Device:Polyfuse -> OOMP:electronic_fuse_0402_resettable
- SW1: symbol Switch:SW_Push -> OOMP:electronic_switch_tactile_surface_mount_xunpu_ts_1088_ar02016
Changed lines of the file:
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@@
   (symbol (lib_id "Device:R") (at 194.31 148.59 270) (unit 1) (body_style 1) (exclude_from_sim no) (in_bom yes) (on_board yes) (in_pos_files yes) (dnp no) (fields_autoplaced yes) (property "Reference" "R6" (at 194.31 144.145 90) (show_name no) (do_not_autoplace no) (effects (font (size 1.27 1.27)))) (property "Value" "2k" (at 194.31 146.685 90) (show_name no) (do_not_autoplace no) (effects (font (size 1.27 1.27)))) (property "Footprint" "Resistor_SMD:R_0402_1005Metric" (at 194.31 146.812 90) (hide yes) (show_name no) (do_not_autoplace no) (effects (font (size 1.27 1.27)))) (property "Datasheet" "" (at 194.31 148.59 0) (hide yes) (show_name no) (do_not_autoplace no) (effects (font (size 1.27 1.27)))) (property "Description" "" (at 194.31 148.59 0) (show_name no) (do_not_autoplace no) (effects (font (size 1.27 1.27)))) (property "LCSC" "C4109" (at 194.31 148.59 0) (hide yes) (show_name no) (do_not_autoplace no) (effects (font (size 1.27 1.27)))) (pin "1") (pin "2") (instances (project "Easyduino_Atmega_Nano" (path "/8ab39f15-d4dc-4110-b18a-e9bac4395ea8" (reference "R6") (unit 1)))))
   (symbol (lib_id "power:PWR_FLAG") (at 48.26 86.36 180) (unit 1) (body_style 1) (exclude_from_sim no) (in_bom yes) (on_board yes) (in_pos_files yes) (dnp no) (fields_autoplaced yes) (property "Reference" "#FLG03" (at 48.26 88.265 0) (hide yes) (show_name no) (do_not_autoplace no) (effects (font (size 1.27 1.27)))) (property "Value" "GND" (at 48.26 91.44 0) (show_name no) (do_not_autoplace no) (effects (font (size 1.27 1.27)))) (property "Footprint" "" (at 48.26 86.36 0) (hide yes) (show_name no) (do_not_autoplace no) (effects (font (size 1.27 1.27)))) (property "Datasheet" "" (at 48.26 86.36 0) (hide yes) (show_name no) (do_not_autoplace no) (effects (font (size 1.27 1.27)))) (property "Description" "Special symbol for telling ERC where power comes from" (at 48.26 86.36 0) (hide yes) (show_name no) (do_not_autoplace no) (effects (font (size 1.27 1.27)))) (pin "1") (instances (project "Easyduino_Atmega_Nano" (path "/8ab39f15-d4dc-4110-b18a-e9bac4395ea8" (reference "#FLG03") (unit 1)))))
-  (symbol (lib_id "Switch:SW_Push") (at 250.19 50.8 0) (unit 1) (body_style 1) (exclude_from_sim no) (in_bom yes) (on_board yes) (in_pos_files yes) (dnp no) (fields_autoplaced yes) (property "Reference" "SW1" (at 250.19 44.45 0) (show_name no) (do_not_autoplace no) (effects (font (size 1.27 1.27)))) (property "Value" "SW_Push" (at 250.19 46.99 0) (show_name no) (do_not_autoplace no) (effects (font (size 1.27 1.27)))) (property "Footprint" "Button_Switch_SMD:SW_Tactile_SPST_NO_Straight_CK_PTS636Sx25SMTRLFS" (at 250.19 45.72 0) (hide yes) (show_name no) (do_not_autoplace no) (effects (font (size 1.27 1.27)))) (property "Datasheet" "" (at 250.19 45.72 0) (hide yes) (show_name no) (do_not_autoplace no) (effects (font (size 1.27 1.27)))) (property "Description" "" (at 250.19 50.8 0) (show_name no) (do_not_autoplace no) (effects (font (size 1.27 1.27)))) (property "LCSC" "C520860" (at 250.19 50.8 0) (hide yes) (show_name no) (do_not_autoplace no) (effects (font (size 1.27 1.27)))) (pin "1") (pin "2") (instances (project "Easyduino_Atmega_Nano" (path "/8ab39f15-d4dc-4110-b18a-e9bac4395ea8" (reference "SW1") (unit 1)))))
-  (symbol (lib_id "Device:Polyfuse") (at 67.31 45.72 90) (unit 1) (body_style 1) (exclude_from_sim no) (in_bom yes) (on_board yes) (in_pos_files yes) (dnp no) (fields_autoplaced yes) (property "Reference" "F1" (at 67.31 40.005 90) (show_name no) (do_not_autoplace no) (effects (font (size 1.27 1.27)))) (property "Value" "Polyfuse" (at 67.31 42.545 90) (show_name no) (do_not_autoplace no) (effects (font (size 1.27 1.27)))) (property "Footprint" "Fuse:Fuse_0402_1005Metric" (at 72.39 44.45 0) (hide yes) (show_name no) (do_not_autoplace no) (effects (font (size 1.27 1.27)) (justify left))) (property "Datasheet" "" (at 67.31 45.72 0) (hide yes) (show_name no) (do_not_autoplace no) (effects (font (size 1.27 1.27)))) (property "Description" "" (at 67.31 45.72 0) (show_name no) (do_not_autoplace no) (effects (font (size 1.27 1.27)))) (property "LCSC" "C914087" (at 67.31 45.72 0) (hide yes) (show_name no) (do_not_autoplace no) (effects (font (size 1.27 1.27)))) (pin "1") (pin "2") (instances (project "Easyduino_Atmega_Nano" (path "/8ab39f15-d4dc-4110-b18a-e9bac4395ea8" (reference "F1") (unit 1)))))
+  (symbol (lib_id "OOMP:electronic_switch_tactile_surface_mount_xunpu_ts_1088_ar02016") (at 250.19 50.8 0) (unit 1) (body_style 1) (exclude_from_sim no) (in_bom yes) (on_board yes) (in_pos_files yes) (dnp no) (fields_autoplaced yes) (property "Reference" "SW1" (at 250.19 44.45 0) (show_name no) (do_not_autoplace no) (effects (font (size 1.27 1.27)))) (property "Value" "SW_Push" (at 250.19 46.99 0) (show_name no) (do_not_autoplace no) (effects (font (size 1.27 1.27)))) (property "Footprint" "Button_Switch_SMD:SW_Tactile_SPST_NO_Straight_CK_PTS636Sx25SMTRLFS" (at 250.19 45.72 0) (hide yes) (show_name no) (do_not_autoplace no) (effects (font (size 1.27 1.27)))) (property "Datasheet" "" (at 250.19 45.72 0) (hide yes) (show_name no) (do_not_autoplace no) (effects (font (size 1.27 1.27)))) (property "Description" "" (at 250.19 50.8 0) (show_name no) (do_not_autoplace no) (effects (font (size 1.27 1.27)))) (property "LCSC" "C520860" (at 250.19 50.8 0) (hide yes) (show_name no) (do_not_autoplace no) (effects (font (size 1.27 1.27)))) (pin "1") (pin "2") (instances (project "Easyduino_Atmega_Nano" (path "/8ab39f15-d4dc-4110-b18a-e9bac4395ea8" (reference "SW1") (unit 1)))))
+  (symbol (lib_id "OOMP:electronic_fuse_0402_resettable") (at 67.31 45.72 90) (unit 1) (body_style 1) (exclude_from_sim no) (in_bom yes) (on_board yes) (in_pos_files yes) (dnp no) (fields_autoplaced yes) (property "Reference" "F1" (at 67.31 40.005 90) (show_name no) (do_not_autoplace no) (effects (font (size 1.27 1.27)))) (property "Value" "Polyfuse" (at 67.31 42.545 90) (show_name no) (do_not_autoplace no) (effects (font (size 1.27 1.27)))) (property "Footprint" "OOMP_MachineSolder:electronic_fuse_0402_resettable" (at 72.39 44.45 0) (hide yes) (show_name no) (do_not_autoplace no) (effects (font (size 1.27 1.27)) (justify left))) (property "Datasheet" "" (at 67.31 45.72 0) (hide yes) (show_name no) (do_not_autoplace no) (effects (font (size 1.27 1.27)))) (property "Description" "" (at 67.31 45.72 0) (show_name no) (do_not_autoplace no) (effects (font (size 1.27 1.27)))) (property "LCSC" "C914087" (at 67.31 45.72 0) (hide yes) (show_name no) (do_not_autoplace no) (effects (font (size 1.27 1.27)))) (pin "1") (pin "2") (instances (project "Easyduino_Atmega_Nano" (path "/8ab39f15-d4dc-4110-b18a-e9bac4395ea8" (reference "F1") (unit 1)))))
   (symbol (lib_id "Device:D_Schottky") (at 66.04 143.51 180) (unit 1) (body_style 1) (exclude_from_sim no) (in_bom yes) (on_board yes) (in_pos_files yes) (dnp no) (fields_autoplaced yes) (property "Reference" "D2" (at 66.3575 137.795 0) (show_name no) (do_not_autoplace no) (effects (font (size 1.27 1.27)))) (property "Value" "D_Schottky" (at 66.3575 140.335 0) (show_name no) (do_not_autoplace no) (effects (font (size 1.27 1.27)))) (property "Footprint" "Diode_SMD:D_0402_1005Metric" (at 66.04 143.51 0) (hide yes) (show_name no) (do_not_autoplace no) (effects (font (size 1.27 1.27)))) (property "Datasheet" "" (at 66.04 143.51 0) (hide yes) (show_name no) (do_not_autoplace no) (effects (font (size 1.27 1.27)))) (property "Description" "" (at 66.04 143.51 0) (show_name no) (do_not_autoplace no) (effects (font (size 1.27 1.27)))) (property "LCSC" "C2837790" (at 66.04 143.51 0) (hide yes) (show_name no) (do_not_autoplace no) (effects (font (size 1.27 1.27)))) (pin "1") (pin "2") (instances (project "Easyduino_Atmega_Nano" (path "/8ab39f15-d4dc-4110-b18a-e9bac4395ea8" (reference "D2") (unit 1)))))
   (symbol (lib_id "Device:C") (at 102.87 39.37 0) (unit 1) (body_style 1) (exclude_from_sim no) (in_bom yes) (on_board yes) (in_pos_files yes) (dnp no) (property "Reference" "C2" (at 101.6 29.845 0) (show_name no) (do_not_autoplace no) (effects (font (size 1.27 1.27)) (justify left))) (property "Value" "100n" (at 101.6 32.385 0) (show_name no) (do_not_autoplace no) (effects (font (size 1.27 1.27)) (justify left))) (property "Footprint" "Capacitor_SMD:C_0402_1005Metric" (at 103.8352 43.18 0) (hide yes) (show_name no) (do_not_autoplace no) (effects (font (size 1.27 1.27)))) (property "Datasheet" "" (at 102.87 39.37 0) (hide yes) (show_name no) (do_not_autoplace no) (effects (font (size 1.27 1.27)))) (property "Description" "" (at 102.87 39.37 0) (show_name no) (do_not_autoplace no) (effects (font (size 1.27 1.27)))) (property "LCSC" "C1525" (at 102.87 39.37 0) (hide yes) (show_name no) (do_not_autoplace no) (effects (font (size 1.27 1.27)))) (pin "1") (pin "2") (instances (project "Easyduino_Atmega_Nano" (path "/8ab39f15-d4dc-4110-b18a-e9bac4395ea8" (reference "C2") (unit 1)))))

Commit message: working
Parts:
- D1, D3: footprint OOMP_MachineSolder:electronic_led_0402 -> LED_SMD:LED_0402_1005Metric; symbol OOMP:electronic_led_0402 -> OOMP:electronic_led_0402_blue
- D2: symbol Device:D_Schottky -> OOMP:electronic_diode_schottky_0402
- F1: footprint OOMP_MachineSolder:electronic_fuse_0402_resettable -> Fuse:Fuse_0402_1005Metric
- J2: symbol Connector_Generic:Conn_02x03_Odd_Even -> OOMP:electronic_connector_header_2_54_mm_pitch_through_hole_dual_row_6_pin
- U1: symbol MCU_Microchip_ATmega:ATmega328P-A -> OOMP:electronic_ic_tqfp_32_7_mm_x_7_mm_microcontroller_8_bit_avr_microchip_atmega328p_au
- U2: symbol Regulator_Linear:XC6206PxxxMR -> OOMP:electronic_ic_sot_23_power_management_linear_voltage_regulator_5_volt_torex_xc6206p502mr
- U3: symbol Interface_USB:CP2102N-Axx-xQFN28 -> OOMP:electronic_ic_qfn_28_5_mm_x_5_mm_converter_usb_to_serial_converter_silicon_labs_cp2102n_a01_gqfn28r
