File: parts/oomp_project_github_hanqaqa_easyduino_atmega328p_arduino_uno_current/data/oomp_design/Easyduino_Atmega.kicad_pcb (KiCad board)
At the start: 4 copper layers, 68.8 x 53.6 mm, 38 parts, among them J1 USB_C_Receptacle_USB2.0, J2 Conn_01x02_Pin, J3 ICSP, SW1 SW_Push, U1 CH340C, U2 ATmega328P-A, U3 AMS1117-5V, U4 AMS1117-3.3V, Y1 16MHz

Commit message: current
Parts:
- D2, D3: footprint Diode_SMD:D_SOD-123 -> OOMP_MachineSolder:electronic_diode_schottky_sod_123_ss14
- F1: footprint Fuse:Fuse_1206_3216Metric -> OOMP_MachineSolder:electronic_fuse_1206_resettable

Commit message: working
Parts:
- C1, C2, C3, C4, C5, C6, C7: footprint OOMP_MachineSolder:electronic_capacitor_0603_100_nano_farad -> Capacitor_SMD:C_0603_1608Metric
- C8, C9: footprint OOMP_MachineSolder:electronic_capacitor_0603_22_pico_farad -> Capacitor_SMD:C_0603_1608Metric
- D2, D3: footprint OOMP_MachineSolder:electronic_diode_schottky_sod_123_ss14 -> Diode_SMD:D_SOD-123
- F1: footprint OOMP_MachineSolder:electronic_fuse_1206_resettable -> Fuse:Fuse_1206_3216Metric
- J2: footprint OOMP_MachineSolder:electronic_connector_header_2_54_mm_pitch_through_hole_2_pin -> Connector_PinHeader_2.54mm:PinHeader_1x02_P2.54mm_Vertical
- R1, R2, R3, R4: footprint OOMP_MachineSolder:electronic_resistor_0603_5100_ohm -> Resistor_SMD:R_0603_1608Metric
- R5: footprint OOMP_MachineSolder:electronic_resistor_0603_330_ohm -> Resistor_SMD:R_0603_1608Metric
- R6, R7: footprint OOMP_MachineSolder:electronic_resistor_0603_2000_ohm -> Resistor_SMD:R_0603_1608Metric
