File: parts/oomp_project_github_hanqaqa_easyduino_atmega328p_arduino_uno_current/data/oomp_design/Easyduino_Atmega.kicad_sch (KiCad schematic)
At the start: 38 parts, among them J1 USB_C_Receptacle_USB2.0, J2 Conn_01x02_Pin, J3 ICSP, SW1 SW_Push, U1 CH340C, U2 ATmega328P-A, U3 AMS1117-5V, U4 AMS1117-3.3V, Y1 16MHz

Commit message: changes
Parts:
- Y1: symbol Device:Crystal_GND24 -> OOMP:electronic_crystal_3225_surface_mount_4_pin_16_mhz_20_pf
Changed lines of the file:
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@@
   (symbol (lib_id "Device:C") (at 179.07 45.72 180) (unit 1) (body_style 1) (exclude_from_sim no) (in_bom yes) (on_board yes) (in_pos_files yes) (dnp no) (property "Reference" "C3" (at 177.165 37.465 0) (show_name no) (do_not_autoplace no) (effects (font (size 1.27 1.27)) (justify right))) (property "Value" "100n" (at 176.53 40.005 0) (show_name no) (do_not_autoplace no) (effects (font (size 1.27 1.27)) (justify right))) (property "Footprint" "Capacitor_SMD:C_0603_1608Metric" (at 178.1048 41.91 0) (hide yes) (show_name no) (do_not_autoplace no) (effects (font (size 1.27 1.27)))) (property "Datasheet" "" (at 179.07 45.72 0) (hide yes) (show_name no) (do_not_autoplace no) (effects (font (size 1.27 1.27)))) (property "Description" "" (at 179.07 45.72 0) (show_name no) (do_not_autoplace no) (effects (font (size 1.27 1.27)))) (property "LCSC" "C14663" (at 179.07 45.72 0) (hide yes) (show_name no) (do_not_autoplace no) (effects (font (size 1.27 1.27)))) (pin "1") (pin "2") (instances (project "Easyduino_Atmega" (path "/e6a7d6e0-1c9e-4c5d-a12b-6a207a6f6562" (reference "C3") (unit 1)))))
   (symbol (lib_id "power:+3.3V") (at 62.23 176.53 0) (unit 1) (body_style 1) (exclude_from_sim no) (in_bom yes) (on_board yes) (in_pos_files yes) (dnp no) (fields_autoplaced yes) (property "Reference" "#PWR033" (at 62.23 180.34 0) (hide yes) (show_name no) (do_not_autoplace no) (effects (font (size 1.27 1.27)))) (property "Value" "+3.3V" (at 62.23 172.72 0) (show_name no) (do_not_autoplace no) (effects (font (size 1.27 1.27)))) (property "Footprint" "" (at 62.23 176.53 0) (hide yes) (show_name no) (do_not_autoplace no) (effects (font (size 1.27 1.27)))) (property "Datasheet" "" (at 62.23 176.53 0) (hide yes) (show_name no) (do_not_autoplace no) (effects (font (size 1.27 1.27)))) (property "Description" "" (at 62.23 176.53 0) (show_name no) (do_not_autoplace no) (effects (font (size 1.27 1.27)))) (pin "1") (instances (project "Easyduino_Atmega" (path "/e6a7d6e0-1c9e-4c5d-a12b-6a207a6f6562" (reference "#PWR033") (unit 1)))))
-  (symbol (lib_id "Device:Crystal_GND24") (at 248.92 88.9 0) (unit 1) (body_style 1) (exclude_from_sim no) (in_bom yes) (on_board yes) (in_pos_files yes) (dnp no) (property "Reference" "Y1" (at 265.43 85.09 0) (show_name no) (do_not_autoplace no) (effects (font (size 1.27 1.27)))) (property "Value" "16MHz" (at 265.43 87.63 0) (show_name no) (do_not_autoplace no) (effects (font (size 1.27 1.27)))) (property "Footprint" "Crystal:Crystal_SMD_3225-4Pin_3.2x2.5mm" (at 248.92 88.9 0) (hide yes) (show_name no) (do_not_autoplace no) (effects (font (size 1.27 1.27)))) (property "Datasheet" "" (at 248.92 88.9 0) (hide yes) (show_name no) (do_not_autoplace no) (effects (font (size 1.27 1.27)))) (property "Description" "Four pin crystal, GND on pins 2 and 4" (at 248.92 88.9 0) (show_name no) (do_not_autoplace no) (effects (font (size 1.27 1.27)))) (property "LCSC" "C13738" (at 248.92 88.9 0) (hide yes) (show_name no) (do_not_autoplace no) (effects (font (size 1.27 1.27)))) (pin "1") (pin "2") (pin "3") (pin "4") (instances (project "Easyduino_Atmega" (path "/e6a7d6e0-1c9e-4c5d-a12b-6a207a6f6562" (reference "Y1") (unit 1)))))
+  (symbol (lib_id "OOMP:electronic_crystal_3225_surface_mount_4_pin_16_mhz_20_pf") (at 248.92 88.9 0) (unit 1) (body_style 1) (exclude_from_sim no) (in_bom yes) (on_board yes) (in_pos_files yes) (dnp no) (property "Reference" "Y1" (at 265.43 85.09 0) (show_name no) (do_not_autoplace no) (effects (font (size 1.27 1.27)))) (property "Value" "16MHz" (at 265.43 87.63 0) (show_name no) (do_not_autoplace no) (effects (font (size 1.27 1.27)))) (property "Footprint" "Crystal:Crystal_SMD_3225-4Pin_3.2x2.5mm" (at 248.92 88.9 0) (hide yes) (show_name no) (do_not_autoplace no) (effects (font (size 1.27 1.27)))) (property "Datasheet" "" (at 248.92 88.9 0) (hide yes) (show_name no) (do_not_autoplace no) (effects (font (size 1.27 1.27)))) (property "Description" "Four pin crystal, GND on pins 2 and 4" (at 248.92 88.9 0) (show_name no) (do_not_autoplace no) (effects (font (size 1.27 1.27)))) (property "LCSC" "C13738" (at 248.92 88.9 0) (hide yes) (show_name no) (do_not_autoplace no) (effects (font (size 1.27 1.27)))) (pin "1") (pin "2") (pin "3") (pin "4") (instances (project "Easyduino_Atmega" (path "/e6a7d6e0-1c9e-4c5d-a12b-6a207a6f6562" (reference "Y1") (unit 1)))))
   (symbol (lib_id "Device:C_Polarized") (at 62.23 148.59 0) (unit 1) (body_style 1) (exclude_from_sim no) (in_bom yes) (on_board yes) (in_pos_files yes) (dnp no) (fields_autoplaced yes) (property "Reference" "C11" (at 65.405 147.066 0) (show_name no) (do_not_autoplace no) (effects (font (size 1.27 1.27)) (justify left))) (property "Value" "22u" (at 65.405 149.606 0) (show_name no) (do_not_autoplace no) (effects (font (size 1.27 1.27)) (justify left))) (property "Footprint" "Capacitor_Tantalum_SMD:CP_EIA-3216-10_Kemet-I" (at 63.1952 152.4 0) (hide yes) (show_name no) (do_not_autoplace no) (effects (font (size 1.27 1.27)))) (property "Datasheet" "" (at 62.23 148.59 0) (hide yes) (show_name no) (do_not_autoplace no) (effects (font (size 1.27 1.27)))) (property "Description" "" (at 62.23 148.59 0) (show_name no) (do_not_autoplace no) (effects (font (size 1.27 1.27)))) (property "LCSC" "C11366" (at 62.23 148.59 0) (hide yes) (show_name no) (do_not_autoplace no) (effects (font (size 1.27 1.27)))) (pin "1") (pin "2") (instances (project "Easyduino_Atmega" (path "/e6a7d6e0-1c9e-4c5d-a12b-6a207a6f6562" (reference "C11") (unit 1)))))
   (symbol (lib_id "OOMP:electronic_led_0603") (at 212.09 147.32 180) (unit 1) (body_style 1) (exclude_from_sim no) (in_bom yes) (on_board yes) (in_pos_files yes) (dnp no) (fields_autoplaced yes) (property "Reference" "D4" (at 213.6775 140.97 0) (show_name no) (do_not_autoplace no) (effects (font (size 1.27 1.27)))) (property "Value" "LED" (at 213.6775 143.51 0) (show_name no) (do_not_autoplace no) (effects (font (size 1.27 1.27)))) (property "Footprint" "Diode_SMD:D_0603_1608Metric" (at 212.09 147.32 0) (hide yes) (show_name no) (do_not_autoplace no) (effects (font (size 1.27 1.27)))) (property "Datasheet" "" (at 212.09 147.32 0) (hide yes) (show_name no) (do_not_autoplace no) (effects (font (size 1.27 1.27)))) (property "Description" "Light emitting diode" (at 212.09 147.32 0) (hide yes) (show_name no) (do_not_autoplace no) (effects (font (size 1.27 1.27)))) (property "LCSC" "C72043" (at 212.09 147.32 0) (hide yes) (show_name no) (do_not_autoplace no) (effects (font (size 1.27 1.27)))) (pin "1") (pin "2") (instances (project "Easyduino_Atmega" (path "/e6a7d6e0-1c9e-4c5d-a12b-6a207a6f6562" (reference "D4") (unit 1)))))

Commit message: current
Parts:
- C10, C11, C12: symbol Device:C_Polarized -> OOMP:electronic_capacitor_3216_avx_a_tantalum_22_micro_farad_10_volt
- D2, D3: footprint Diode_SMD:D_SOD-123 -> OOMP_MachineSolder:electronic_diode_schottky_sod_123_ss14; symbol Device:D_Schottky -> OOMP:electronic_diode_schottky_sod_123_ss14
- F1: footprint Fuse:Fuse_1206_3216Metric -> OOMP_MachineSolder:electronic_fuse_1206_resettable; symbol Device:Polyfuse -> OOMP:electronic_fuse_1206_resettable

Commit message: working
Parts:
- D2, D3: footprint OOMP_MachineSolder:electronic_diode_schottky_sod_123_ss14 -> Diode_SMD:D_SOD-123
- F1: footprint OOMP_MachineSolder:electronic_fuse_1206_resettable -> Fuse:Fuse_1206_3216Metric
- J3: symbol Connector_Generic:Conn_02x03_Odd_Even -> OOMP:electronic_connector_header_2_54_mm_pitch_through_hole_dual_row_6_pin
- L1: symbol Device:L -> OOMP:electronic_inductor_0603_10_micro_henry
- U2: symbol MCU_Microchip_ATmega:ATmega328P-A -> OOMP:electronic_ic_tqfp_32_7_mm_x_7_mm_microcontroller_8_bit_avr_microchip_atmega328p_au

Commit message: working
Parts:
- D1: symbol Power_Protection:PRTR5V0U2X -> OOMP:electronic_diode_tvs_array_sot_143_nxp_prtr5v0u2x
- SW1: symbol Switch:SW_Push -> OOMP:electronic_switch_tactile_surface_mount_omron_b3fs_100xp
