File: parts/oomp_project_github_hanqaqa_easyduino_esp32_current/data/oomp_design/Easyduino_ESP32.kicad_pcb (KiCad board)
At the start: 4 copper layers, 28.4 x 47.9 mm, 29 parts, among them J1 USB_C_Receptacle_USB2.0, Q1 SS8050, Q2 SS8050, SW1 SW_Push, SW2 SW_Push, U1 CP2102N-Axx-xQFN28, U2 ESP32-WROOM-E, U3 AMS1117-3.3, U4 ESP32-DevKitC

Commit message: changes
Parts:
- D1: footprint Package_TO_SOT_SMD:SOT-143 -> OOMP_MachineSolder:electronic_diode_tvs_array_sot_143_littelfuse_sp0503bahtg
- D2: footprint OOMP_MachineSolder:electronic_led_0402 -> OOMP_MachineSolder:electronic_led_0402_blue
- Q1, Q2: footprint Package_TO_SOT_SMD:SOT-23W -> OOMP_MachineSolder:electronic_transistor_sot_23_bipolar_npn_25_volt_1_5_amp_jsmsemi_ss8050
- U3: footprint Package_TO_SOT_SMD:SOT-223-3_TabPin2 -> OOMP_MachineSolder:electronic_ic_sot_223_3_power_management_linear_voltage_regulator_3_3_volt_advanced_monolithic_syste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

Commit message: working
Parts:
- C1: footprint OOMP_MachineSolder:electronic_capacitor_0402_1_micro_farad -> Capacitor_SMD:C_0402_1005Metric
- C10, C2, C3, C4, C6, C9: footprint OOMP_MachineSolder:electronic_capacitor_0402_100_nano_farad -> Capacitor_SMD:C_0402_1005Metric
- D1: footprint OOMP_MachineSolder:electronic_diode_tvs_array_sot_143_littelfuse_sp0503bahtg -> Package_TO_SOT_SMD:SOT-143
- D2: footprint OOMP_MachineSolder:electronic_led_0402_blue -> LED_SMD:LED_0402_1005Metric
- Q1, Q2: footprint OOMP_MachineSolder:electronic_transistor_sot_23_bipolar_npn_25_volt_1_5_amp_jsmsemi_ss8050 -> Package_TO_SOT_SMD:SOT-23W
- R1, R4, R5, R7: footprint OOMP_MachineSolder:electronic_resistor_0402_10000_ohm -> Resistor_SMD:R_0402_1005Metric
- R2, R3, R8: footprint OOMP_MachineSolder:electronic_resistor_0402_5100_ohm -> Resistor_SMD:R_0402_1005Metric
- R6: footprint OOMP_MachineSolder:electronic_resistor_0402_2000_ohm -> Resistor_SMD:R_0402_1005Metric
- U3: footprint OOMP_MachineSolder:electronic_ic_sot_223_3_power_management_linear_voltage_regulator_3_3_volt_advanced_monolithic_syste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 -> Package_TO_SOT_SMD:SOT-223-3_TabPin2
