File: parts/oomp_project_github_hanqaqa_easyduino_esp32_current/data/oomp_design/Easyduino_ESP32.kicad_sch (KiCad schematic)
At the start: 29 parts, among them J1 USB_C_Receptacle_USB2.0, Q1 SS8050, Q2 SS8050, SW1 SW_Push, SW2 SW_Push, U1 CP2102N-Axx-xQFN28, U2 ESP32-WROOM-E, U3 AMS1117-3.3, U4 ESP32-DevKitC

Commit message: changes
Parts:
- C5, C7, C8: symbol Device:C_Polarized -> OOMP:electronic_capacitor_3216_avx_a_tantalum_22_micro_farad_10_volt
- D1: footprint Package_TO_SOT_SMD:SOT-143 -> OOMP_MachineSolder:electronic_diode_tvs_array_sot_143_littelfuse_sp0503bahtg; symbol Power_Protection:SP0503BAHT -> OOMP:electronic_diode_tvs_array_sot_143_littelfuse_sp0503bahtg
- D2: footprint OOMP_MachineSolder:electronic_led_0402 -> OOMP_MachineSolder:electronic_led_0402_blue; symbol OOMP:electronic_led_0402 -> OOMP:electronic_led_0402_blue
- SW1, SW2: symbol Switch:SW_Push -> OOMP:electronic_switch_tactile_surface_mount_xunpu_ts_1088_ar02016
- U3: footprint Package_TO_SOT_SMD:SOT-223-3_TabPin2 -> OOMP_MachineSolder:electronic_ic_sot_223_3_power_management_linear_voltage_regulator_3_3_volt_advanced_monolithic_syste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; symbol Regulator_Linear:AMS1117-3.3 -> OOMP:electronic_ic_sot_223_3_power_management_linear_voltage_regulator_3_3_volt_advanced_monolithic_systems_ams1117_3_3

Commit message: working
Parts:
- D1: footprint OOMP_MachineSolder:electronic_diode_tvs_array_sot_143_littelfuse_sp0503bahtg -> Package_TO_SOT_SMD:SOT-143
- D2: footprint OOMP_MachineSolder:electronic_led_0402_blue -> LED_SMD:LED_0402_1005Metric
- U1: symbol Interface_USB:CP2102N-Axx-xQFN28 -> OOMP:electronic_ic_qfn_28_5_mm_x_5_mm_converter_usb_to_serial_converter_silicon_labs_cp2102n_a01_gqfn28r
- U3: footprint OOMP_MachineSolder:electronic_ic_sot_223_3_power_management_linear_voltage_regulator_3_3_volt_advanced_monolithic_syste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 -> Package_TO_SOT_SMD:SOT-223-3_TabPin2
