File: parts/oomp_project_github_hanqaqa_easyduino_esp32s3_current/data/oomp_design/Easyduino_ESP32S3.kicad_sch (KiCad schematic)
At the start: 35 parts, among them J1 USB_C_Receptacle_USB2.0, J2 USB_C_Receptacle_USB2.0, Q1 Q_NPN_BCE, Q2 Q_NPN_BCE, SW1 SW_Push, SW2 SW_Push, U1 ESP32-S3-WROOM-1, U2 ESP32-S3-DevKitC, U3 CP2102N-Axx-xQFN28, U5 AMS1117-3.3

Commit message: current
Parts:
- C10, C6, C7: symbol Device:C_Polarized -> OOMP:electronic_capacitor_3216_avx_a_tantalum_22_micro_farad_10_volt
- SW1, SW2: symbol Switch:SW_Push -> OOMP:electronic_switch_tactile_surface_mount_xunpu_ts_1088_ar02016

Commit message: working
Parts:
- D1: symbol OOMP:electronic_led_0402 -> OOMP:electronic_led_0402_blue
- D2, D3: symbol Device:D_Schottky -> OOMP:electronic_diode_schottky_0402
- D4: footprint OOMP_MachineSolder:electronic_led_0402 -> LED_SMD:LED_0402_1005Metric; symbol OOMP:electronic_led_0402 -> OOMP:electronic_led_0402_blue
- U3: symbol Interface_USB:CP2102N-Axx-xQFN28 -> OOMP:electronic_ic_qfn_28_5_mm_x_5_mm_converter_usb_to_serial_converter_silicon_labs_cp2102n_a01_gqfn28r
- U5: symbol Regulator_Linear:AMS1117-3.3 -> OOMP:electronic_ic_sot_223_3_power_management_linear_voltage_regulator_3_3_volt_advanced_monolithic_systems_ams1117_3_3
