File: parts/oomp_project_github_dangerousprototypes_buspirate5_hardware_5_rev10a/data/oomp_design/micro-rp2040.kicad_sch (KiCad schematic)
At the start: 38 parts, among them J201 Conn_01x03, J202 TYPE-C-31-M-12, SW101 SW_SPST, SW102 4P_button_sw, U102 W25Q128JVSIQ, U103 RP2040, U105 MT29F1G01ABAFDWB, U401 ME6211A33PG-N, Y101 12Mhz

Commit message: working
Parts:
- SW101: symbol Switch:SW_SPST -> OOMP:electronic_switch_tactile_surface_mount_pts810
Changed lines of the file:
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@@
   (symbol (lib_id "Device:C_Small") (at 209.55 43.18 0) (unit 1) (in_bom yes) (on_board yes) (dnp no) (property "Reference" "C109" (at 214.63 41.91 0) (effects (font (size 1.27 1.27)))) (property "Value" "2.2uF" (at 214.63 44.45 0) (effects (font (size 1.27 1.27)))) (property "Footprint" "Capacitor_SMD:C_0402_1005Metric" (at 209.55 43.18 0) (effects (font (size 1.27 1.27)) hide)) (property "Datasheet" "~" (at 209.55 43.18 0) (effects (font (size 1.27 1.27)) hide)) (property "RMB" "0.043101" (at 209.55 43.18 0) (effects (font (size 1.27 1.27)) hide)) (property "Supplier" "https://item.szlcsc.com/108589.html" (at 209.55 43.18 0) (effects (font (size 1.27 1.27)) hide)) (pin "1") (pin "2") (instances (project "BusPirate-5-rev10" (path "/1f56410a-eaac-4444-b0f7-cfd3531e22ac/00000000-0000-0000-0000-000060c8ec36" (reference "C109") (unit 1)))))
   (symbol (lib_id "power:GND") (at 209.55 45.72 0) (unit 1) (in_bom yes) (on_board yes) (dnp no) (property "Reference" "#PWR0123" (at 209.55 52.07 0) (effects (font (size 1.27 1.27)) hide)) (property "Value" "GND" (at 209.677 50.1142 0) (effects (font (size 1.27 1.27)))) (property "Footprint" "" (at 209.55 45.72 0) (effects (font (size 1.27 1.27)) hide)) (property "Datasheet" "" (at 209.55 45.72 0) (effects (font (size 1.27 1.27)) hide)) (pin "1") (instances (project "BusPirate-5-rev10" (path "/1f56410a-eaac-4444-b0f7-cfd3531e22ac/00000000-0000-0000-0000-000060c8ec36" (reference "#PWR0123") (unit 1)))))
-  (symbol (lib_id "Switch:SW_SPST") (at 73.66 111.76 0) (unit 1) (in_bom yes) (on_board yes) (dnp no) (property "Reference" "SW101" (at 73.66 105.791 0) (effects (font (size 1.27 1.27)))) (property "Value" "SW_SPST" (at 73.66 108.1024 0) (effects (font (size 1.27 1.27)))) (property "Footprint" "Button_Switch_SMD:SW_SPST_PTS810" (at 73.66 111.76 0) (effects (font (size 1.27 1.27)) hide)) (property "Datasheet" "~" (at 73.66 111.76 0) (effects (font (size 1.27 1.27)) hide)) (pin "1") (pin "2") (instances (project "BusPirate-5-rev10" (path "/1f56410a-eaac-4444-b0f7-cfd3531e22ac/00000000-0000-0000-0000-000060c8ec36" (reference "SW101") (unit 1)))))
+  (symbol (lib_id "OOMP:electronic_switch_tactile_surface_mount_pts810") (at 73.66 111.76 0) (unit 1) (in_bom yes) (on_board yes) (dnp no) (property "Reference" "SW101" (at 73.66 105.791 0) (effects (font (size 1.27 1.27)))) (property "Value" "SW_SPST" (at 73.66 108.1024 0) (effects (font (size 1.27 1.27)))) (property "Footprint" "Button_Switch_SMD:SW_SPST_PTS810" (at 73.66 111.76 0) (effects (font (size 1.27 1.27)) hide)) (property "Datasheet" "~" (at 73.66 111.76 0) (effects (font (size 1.27 1.27)) hide)) (pin "1") (pin "2") (instances (project "BusPirate-5-rev10" (path "/1f56410a-eaac-4444-b0f7-cfd3531e22ac/00000000-0000-0000-0000-000060c8ec36" (reference "SW101") (unit 1)))))
   (symbol (lib_id "OOMP:electronic_resistor_0402_1000_ohm") (at 68.58 107.95 0) (unit 1) (in_bom yes) (on_board yes) (dnp no) (property "Reference" "R101" (at 66.04 106.68 0) (effects (font (size 1.27 1.27)))) (property "Value" "1K" (at 66.04 109.22 0) (effects (font (size 1.27 1.27)))) (property "Footprint" "Resistor_SMD:R_0402_1005Metric" (at 68.58 107.95 0) (effects (font (size 1.27 1.27)) hide)) (property "Datasheet" "~" (at 68.58 107.95 0) (effects (font (size 1.27 1.27)) hide)) (property "RMB" "0.006373" (at 68.58 107.95 0) (effects (font (size 1.27 1.27)) hide)) (property "Supplier" "https://item.szlcsc.com/116008.html" (at 68.58 107.95 0) (effects (font (size 1.27 1.27)) hide)) (pin "1") (pin "2") (instances (project "BusPirate-5-rev10" (path "/1f56410a-eaac-4444-b0f7-cfd3531e22ac/00000000-0000-0000-0000-000060c8ec36" (reference "R101") (unit 1)))))
   (symbol (lib_id "power:GND") (at 78.74 111.76 0) (unit 1) (in_bom yes) (on_board yes) (dnp no) (property "Reference" "#PWR0110" (at 78.74 118.11 0) (effects (font (size 1.27 1.27)) hide)) (property "Value" "GND" (at 78.867 116.1542 0) (effects (font (size 1.27 1.27)))) (property "Footprint" "" (at 78.74 111.76 0) (effects (font (size 1.27 1.27)) hide)) (property "Datasheet" "" (at 78.74 111.76 0) (effects (font (size 1.27 1.27)) hide)) (pin "1") (instances (project "BusPirate-5-rev10" (path "/1f56410a-eaac-4444-b0f7-cfd3531e22ac/00000000-0000-0000-0000-000060c8ec36" (reference "#PWR0110") (unit 1)))))
