File: parts/oomp_project_github_adafruit_adafruit_adxl345_pcb_adxl345_stemma_qt_current/data/oomp_design/ADXL345 STEMMA QT.kicad_sch (KiCad schematic)
At the start: 21 parts, among them Q2 BSS138, U1 ADXL343, U2 AP2112K-3.3

Commit message: changes
Parts:
- removed C1: 0.1uF, kicad_file:0603-NO, symbol kicad_file-eagle-import:CAP_CERAMIC0603_NO
- removed C2: 10uF, kicad_file:_0805MP, symbol kicad_file-eagle-import:CAP_CERAMIC_0805MP
- removed C3: 10uF, kicad_file:0805-NO, symbol kicad_file-eagle-import:CAP_CERAMIC0805-NOOUTLINE
- removed CONN3, CONN4: STEMMA_I2C_QT, kicad_file:JST_SH4, symbol kicad_file-eagle-import:STEMMA_I2C_QT
- removed D1: GREEN, kicad_file:CHIPLED_0603_NOOUTLINE, symbol kicad_file-eagle-import:LED0603_NOOUTLINE
- removed D2: 1N4148, kicad_file:SOD-323, symbol kicad_file-eagle-import:DIODESOD-323
- removed FID3, FID4: FIDUCIAL_1MM, kicad_file:FIDUCIAL_1MM, symbol kicad_file-eagle-import:FIDUCIAL_1MM
- removed JP1: HEADER-1X670MIL, kicad_file:1X06_ROUND_70, symbol kicad_file-eagle-import:HEADER-1X670MIL
- removed JP2: HEADER-1X4ROUND, kicad_file:1X04_ROUND, symbol kicad_file-eagle-import:HEADER-1X4ROUND
- removed Q2: BSS138, kicad_file:SOT363, symbol kicad_file-eagle-import:MOSFET-N_DUAL
- removed R1, R3: 10K, kicad_file:RESPACK_4X0603, symbol kicad_file-eagle-import:RESISTOR_4PACK
- removed SJ1: SOLDERJUMPERCLOSED, kicad_file:SOLDERJUMPER_CLOSEDWIRE, symbol kicad_file-eagle-import:SOLDERJUMPERCLOSED
- removed U$1, U$17, U$19, U$21: MOUNTINGHOLE2.5, kicad_file:MOUNTINGHOLE_2.5_PLATED, symbol kicad_file-eagle-import:MOUNTINGHOLE2.5
- removed U1: ADXL343, kicad_file:LGA14, symbol kicad_file-eagle-import:ACCEL_ADXL343
- removed U2: AP2112K-3.3, kicad_file:SOT23-5, symbol kicad_file-eagle-import:VREG_SOT23-5
- added C1: 0.1uF, kicad_file:0603-NO, symbol kicad_file-eagle-import:microbuilder_CAP_CERAMIC0603_NO
- added C2: 10uF, kicad_file:_0805MP, symbol kicad_file-eagle-import:microbuilder_CAP_CERAMIC_0805MP
- added C3: 10uF, kicad_file:0805-NO, symbol kicad_file-eagle-import:microbuilder_CAP_CERAMIC0805-NOOUTLINE
- added CONN3, CONN4: STEMMA_I2C_QT, kicad_file:JST_SH4, symbol kicad_file-eagle-import:microbuilder_STEMMA_I2C_QT
- added D1: GREEN, kicad_file:CHIPLED_0603_NOOUTLINE, symbol kicad_file-eagle-import:microbuilder_LED0603_NOOUTLINE
- added D2: 1N4148, kicad_file:SOD-323, symbol kicad_file-eagle-import:microbuilder_DIODESOD-323
- added FID3, FID4: FIDUCIAL_1MM, kicad_file:FIDUCIAL_1MM, symbol kicad_file-eagle-import:microbuilder_FIDUCIAL_1MM
- added JP1: HEADER-1X670MIL, kicad_file:1X06_ROUND_70, symbol kicad_file-eagle-import:microbuilder_HEADER-1X670MIL
- added JP2: HEADER-1X4ROUND, kicad_file:1X04_ROUND, symbol kicad_file-eagle-import:microbuilder_HEADER-1X4ROUND
- added Q2: BSS138, kicad_file:SOT363, symbol kicad_file-eagle-import:microbuilder_MOSFET-N_DUAL
- added R1, R3: 10K, kicad_file:RESPACK_4X0603, symbol kicad_file-eagle-import:microbuilder_RESISTOR_4PACK
- added SJ1: SOLDERJUMPERCLOSED, kicad_file:SOLDERJUMPER_CLOSEDWIRE, symbol kicad_file-eagle-import:microbuilder_SOLDERJUMPERCLOSED
- added U$1, U$17, U$19, U$21: MOUNTINGHOLE2.5, kicad_file:MOUNTINGHOLE_2.5_PLATED, symbol kicad_file-eagle-import:adafruit_electromech_MOUNTINGHOLE2.5
- added U1: ADXL343, kicad_file:LGA14, symbol kicad_file-eagle-import:microbuilder_ACCEL_ADXL343
- added U2: AP2112K-3.3, kicad_file:SOT23-5, symbol kicad_file-eagle-import:adafruit_power_VREG_SOT23-5
Connections:
- net 3.3V: now also C1.1, C3.1, JP1.2, Q2.2 (G), Q2.5 (G), R1.1, R1.2 (1), R3.2 (1), R3.4 (1), U1.1 (VDD(I/O)), U1.6 (VIN), U2.5 (OUT)
- net CS: now also D2.C, JP2.4
- net CS_3V: now also D2.A, R1.3 (1), R1.6 (2), R1.7 (2), U1.7 (CS)
- net GND: now also C1.2, C2.2, C3.2, CONN3.1 (GND), CONN3.MT1 (MT), CONN3.MT2 (MT), CONN4.1 (GND), CONN4.MT1 (MT), CONN4.MT2 (MT), D1.C, JP1.3, JP2.1, R1.4 (1), U1.2 (GND), U1.4 (GND), U1.5 (GND), U2.2 (GND)
- net INT1: now also JP1.6, U1.8 (INT1)
- net INT2: now also JP2.2, U1.9 (INT2)
- net SCL: now also CONN3.4 (SCL), CONN4.4 (SCL), JP1.4, Q2.6 (D), R3.8 (2)
- net SCL_3V: now also Q2.1 (S), R3.7 (2), U1.14 (SCL)
- net SDA/SDIO: now also CONN3.3 (SDA), CONN4.3 (SDA), JP1.5, Q2.3 (D), R3.6 (2)
- net SDA/SDIO_3V: now also Q2.4 (S), R3.5 (2), U1.13 (SDA)
- net SDO: now also JP2.3, R1.5 (2), U1.12 (ADDR/SDO)
- net VCC: now also C2.1, CONN3.2 (V+), CONN4.2 (V+), JP1.1, R3.1, R3.3 (1), U2.1 (IN), U2.3 (EN)
- new net: D1.A, SJ1.1
- new net: R1.8 (2), SJ1.2
