File: parts/oomp_project_github_adafruit_adafruit_lis3_dh_breakout_pcb_lis3dh_breakout_current/data/oomp_design/Adafruit LIS3DH.kicad_sch (KiCad schematic)
At the start: 21 parts, among them Q2 BSS138, U1 LIS3DHTR, U2 AP2112K-3.3

Commit message: changes
Parts:
- removed C1: 0.1uF, kicad_file:0603-NO, symbol kicad_file-eagle-import:CAP_CERAMIC0603_NO
- removed C2, C3: 10uF, kicad_file:0805-NO, symbol kicad_file-eagle-import:CAP_CERAMIC0805-NOOUTLINE
- removed CONN3, CONN4: STEMMA_I2C_QT, kicad_file:JST_SH4, symbol kicad_file-eagle-import:STEMMA_I2C_QT
- removed D1: GREEN, kicad_file:CHIPLED_0603_NOOUTLINE, symbol kicad_file-eagle-import:LED0603_NOOUTLINE
- removed D2: 1N4148, kicad_file:SOD-323, symbol kicad_file-eagle-import:DIODESOD-323
- removed FID3, FID4: FIDUCIAL_1MM, kicad_file:FIDUCIAL_1MM, symbol kicad_file-eagle-import:FIDUCIAL_1MM
- removed JP2, JP3: HEADER-1X670MIL, kicad_file:1X06_ROUND_70, symbol kicad_file-eagle-import:HEADER-1X670MIL
- removed Q2: BSS138, kicad_file:SOT363, symbol kicad_file-eagle-import:MOSFET-N_DUAL
- removed R1, R3: 10K, kicad_file:RESPACK_4X0603, symbol kicad_file-eagle-import:RESISTOR_4PACK
- removed SJ1: SOLDERJUMPER, kicad_file:SOLDERJUMPER_ARROW_NOPASTE, symbol kicad_file-eagle-import:SOLDERJUMPER
- removed U$1, U$17, U$19, U$21: MOUNTINGHOLE2.5, kicad_file:MOUNTINGHOLE_2.5_PLATED, symbol kicad_file-eagle-import:MOUNTINGHOLE2.5
- removed U1: LIS3DHTR, kicad_file:LGA16_3X3MM, symbol kicad_file-eagle-import:ACCEL_LIS3DHTR
- removed U2: AP2112K-3.3, kicad_file:SOT23-5, symbol kicad_file-eagle-import:VREG_SOT23-5
- added C1: 0.1uF, kicad_file:0603-NO, symbol kicad_file-eagle-import:microbuilder_CAP_CERAMIC0603_NO
- added C2, C3: 10uF, kicad_file:0805-NO, symbol kicad_file-eagle-import:microbuilder_CAP_CERAMIC0805-NOOUTLINE
- added CONN3, CONN4: STEMMA_I2C_QT, kicad_file:JST_SH4, symbol kicad_file-eagle-import:microbuilder_STEMMA_I2C_QT
- added D1: GREEN, kicad_file:CHIPLED_0603_NOOUTLINE, symbol kicad_file-eagle-import:microbuilder_LED0603_NOOUTLINE
- added D2: 1N4148, kicad_file:SOD-323, symbol kicad_file-eagle-import:microbuilder_DIODESOD-323
- added FID3, FID4: FIDUCIAL_1MM, kicad_file:FIDUCIAL_1MM, symbol kicad_file-eagle-import:microbuilder_FIDUCIAL_1MM
- added JP2, JP3: HEADER-1X670MIL, kicad_file:1X06_ROUND_70, symbol kicad_file-eagle-import:microbuilder_HEADER-1X670MIL
- added Q2: BSS138, kicad_file:SOT363, symbol kicad_file-eagle-import:microbuilder_MOSFET-N_DUAL
- added R1, R3: 10K, kicad_file:RESPACK_4X0603, symbol kicad_file-eagle-import:microbuilder_RESISTOR_4PACK
- added SJ1: SOLDERJUMPER, kicad_file:SOLDERJUMPER_ARROW_NOPASTE, symbol kicad_file-eagle-import:microbuilder_SOLDERJUMPER
- added U$1, U$17, U$19, U$21: MOUNTINGHOLE2.5, kicad_file:MOUNTINGHOLE_2.5_PLATED, symbol kicad_file-eagle-import:microbuilder_MOUNTINGHOLE2.5
- added U1: LIS3DHTR, kicad_file:LGA16_3X3MM, symbol kicad_file-eagle-import:microbuilder_ACCEL_LIS3DHTR
- added U2: AP2112K-3.3, kicad_file:SOT23-5, symbol kicad_file-eagle-import:microbuilder_VREG_SOT23-5
Connections:
- net 3.3V: now also C1.1, C3.1, JP3.2, Q2.2 (G), Q2.5 (G), R1.1, R1.5 (2), R1.7 (2), R1.8 (2), R3.2 (1), R3.4 (1), SJ1.1, U1.1 (VDDIO), U1.14 (VDD), U2.5 (OUT)
- net ADC1: now also JP2.3, U1.16 (ADC1)
- net ADC2: now also JP2.4, U1.15 (ADC2)
- net ADC3: now also JP2.5, U1.13 (ADC3)
- net CS: now also D2.C, JP2.1
- net GND: now also C1.2, C2.2, C3.2, CONN3.1 (GND), CONN4.1 (GND), D1.C, JP3.3, R1.6 (2), U1.10 (RES(GND)), U1.12 (GND), U1.5 (GND), U2.2 (GND)
- net INT1: now also JP3.6, U1.11 (INT1)
- net INT2: now also JP2.6, U1.9 (INT2)
- net SCL: now also CONN3.4 (SCL), CONN4.4 (SCL), JP3.4, Q2.6 (D), R3.8 (2)
- net SCL_3V: now also Q2.1 (S), R3.7 (2), U1.4 (SCL)
- net SDA: now also CONN3.3 (SDA), CONN4.3 (SDA), JP3.5, Q2.3 (D), R3.6 (2)
- net SDA_3V: now also Q2.4 (S), R3.5 (2), U1.6 (SDA)
- net SDO: now also JP2.2, R1.3 (1), SJ1.2, U1.7 (SDO)
- net VCC: now also C2.1, CONN3.2 (V+), CONN4.2 (V+), JP3.1, R3.1, R3.3 (1), U2.1 (IN), U2.3 (EN)
- new net: D2.A, R1.2 (1), U1.8 (CS)
- new net: D1.A, R1.4 (1)
